File: pcb/keyboard.kicad_pcb (KiCad board)
At the start: 2 copper layers, 436.8 x 114.6 mm, 438 parts, among them P1 USB_MiniB, P2 Do Not Populate, SW0 ESC, SW1 F1, SW10 F10, SW100 LCTL, SW101 LSPR, SW102 LALT, SW103 SP, SW109 RALT, SW11 F11, SW110 RSPR, SW111 MENU, SW112 RCTL, SW113 LEFT, SW114 DOWN, SW115 RIGHT, SW116 NP-0, SW118 NP-PER, SW12 F12, SW120 SW_P, SW13 BCKSP, SW14 PSCR, SW15 SCLK, SW16 PAUS, SW2 F2, SW20 TILDE, SW21 N1, SW22 N2, SW23 N3, SW24 N4, SW25 N5, SW26 N6, SW27 N7, SW28 N8, SW29 N9, SW3 F3, SW30 N0, SW31 MIN, SW32 EQ, SW33 INS, SW34 HOME, SW35 PGUP, SW36 NP-NMLK, SW37 NP-FWSL, SW38 NP-ASTR, SW39 NP-MNS, SW4 F4, SW40 TAB, SW41 Q, SW42 W, SW43 E, SW44 R, SW45 T, SW46 Y, SW47 U, SW48 I, SW49 O, SW5 F5, SW50 P, SW51 SQBRL, SW52 SQBRR, SW53 DEL, SW54 END, SW55 PGDN, SW56 NP-7, SW57 NP-8, SW58 NP-9, SW59 NP-PLS, SW6 F6, SW60 CPLK, SW61 A, SW62 S, SW63 D, SW64 F, SW65 G, SW66 H, SW67 J, SW68 K, SW69 L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

Commit message: modified:   ../README.md 	modified:   LedReverseMount3_2x1_6mmDialight.pretty/LED Reverse Mount 3.2x1.6mm Dialight.kicad_mod 	new file:   cern_ohl_v_1_2.txt 	new file:   cern_ohl_v_1_2_howto.pdf 	new file:   changes.txt 	new file:   dorkyboard_schematic.pdf 	new file:   gerbers/dorkeyboard-B.Cu.gbr 	new file:   gerbers/dorkeyboard-B.Mask.gbr 	new file:   gerbers/dorkeyboard-B.SilkS.gbr 	new file:   gerbers/dorkeyboard-Edge.Cuts.gbr 	new file:   gerbers/dorkeyboard-F.Cu.gbr 	new file:   gerbers/dorkeyboard-F.Mask.gbr 	new file:   gerbers/dorkeyboard-F.SilkS.gbr 	new file:   gerbers/dorkeyboard-NPTH.drl 	new file:   gerbers/dorkeyboard.drl 	modified:   keyboard.kicad_pcb 	modified:   keyboard.pro 	new file:   product.txt
Parts:
- removed the REF** at (110.0, 225.0)
- removed the REF** at (360.0, 185.0)
- removed the REF** at (370.0, 185.0)
- removed the REF** at (380.0, 185.0)
- removed the REF** at (180.0, 245.0)
Connections:
- U1 pad 45: (no net) -> GND
Routing:
- net /matrix/Row9: track 255.3 -> 254.4 mm
Other:
- net class Default: clearance 0.2 -> 0.16
- rule trace_clearance: 0.2 -> 0.16
